File: Hardware/ProBack_LED_backlight/2xLED_Panel.brd (EAGLE design)
At the start: 48 x 6 mm, 9 parts

Commit message: Update boards and schematic
Parts:
- moved D1 0.70 mm to (15.3, 1.30), turned to 180 degrees
- moved D2 0.70 mm to (31.3, 1.25), turned to 180 degrees
- moved D3 0.70 mm to (15.3, 4.75), turned to 180 degrees
- moved D4 0.70 mm to (31.3, 4.75), turned to 180 degrees
Changed lines of the file:
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@@
 </autorouter>
 <elements>
-<element name="D1" library="Yuji_LED" package="2835_SMD" value="YUJI_2835_SMD" x="16" y="1.25" smashed="yes">
-<attribute name="NAME" x="18.62" y="0.92" size="0.6096" layer="21"/>
+<element name="D1" library="Yuji_LED" package="2835_SMD" value="YUJI_2835_SMD" x="15.3" y="1.3" smashed="yes" rot="R180">
+<attribute name="NAME" x="12.68" y="1.63" size="0.6096" layer="21" rot="R180"/>
 </element>
-<element name="D2" library="Yuji_LED" package="2835_SMD" value="YUJI_2835_SMD" x="32" y="1.25" smashed="yes">
-<attribute name="NAME" x="34.62" y="1.02" size="0.6096" layer="21"/>
+<element name="D2" library="Yuji_LED" package="2835_SMD" value="YUJI_2835_SMD" x="31.3" y="1.25" smashed="yes" rot="R180">
+<attribute name="NAME" x="28.68" y="1.48" size="0.6096" layer="21" rot="R180"/>
 </element>
 <element name="FRAME1" library="SparkFun-Aesthetics" package="CREATIVE_COMMONS" value="FRAME-LEDGER" x="0" y="0" smashed="yes">
@@
 <attribute name="VALUE" x="46.1" y="1.3" size="0.0254" layer="27" rot="R90"/>
 </element>
-<element name="D3" library="Yuji_LED" package="2835_SMD" value="YUJI_2835_SMD" x="16" y="4.75" smashed="yes"/>
-<element name="D4" library="Yuji_LED" package="2835_SMD" value="YUJI_2835_SMD" x="32" y="4.75" smashed="yes"/>
+<element name="D3" library="Yuji_LED" package="2835_SMD" value="YUJI_2835_SMD" x="15.3" y="4.75" smashed="yes" rot="R180"/>
+<element name="D4" library="Yuji_LED" package="2835_SMD" value="YUJI_2835_SMD" x="31.3" y="4.75" smashed="yes" rot="R180"/>
 <element name="+L" library="wirepad" package="2,15/1,0" package3d_urn="urn:adsk.eagle:package:30831/1" value="" x="1.9" y="4.7" smashed="yes">
 <attribute name="POPULARITY" value="11" x="1.9" y="-3.3" size="1.778" layer="27" display="off"/>
@@
 <contactref element="D1" pad="CATHODE"/>
 <contactref element="D2" pad="ANODE"/>
-<wire x1="16.95" y1="1.25" x2="30.7" y2="1.25" width="1.27" layer="1"/>
+<wire x1="30.35" y1="1.25" x2="17.47" y2="1.25" width="1.27" layer="1"/>
+<wire x1="17.47" y1="1.25" x2="16.6" y2="1.3" width="1.27" layer="1"/>
 </signal>
 <signal name="N$2">
 <contactref element="+" pad="1"/>
 <contactref element="D1" pad="ANODE"/>
-<wire x1="1.9" y1="1.3" x2="14.65" y2="1.3" width="1.27" layer="1"/>
-<wire x1="14.65" y1="1.3" x2="14.7" y2="1.25" width="1.27" layer="1"/>
+<wire x1="14.35" y1="1.3" x2="1.9" y2="1.3" width="1.27" layer="1"/>
 </signal>
 <signal name="N$3">
 <contactref element="D2" pad="CATHODE"/>
 <contactref element="-" pad="1"/>
-<wire x1="32.95" y1="1.25" x2="46.05" y2="1.25" width="1.27" layer="1"/>
+<wire x1="32.6" y1="1.25" x2="46.05" y2="1.25" width="1.27" layer="1"/>
 <wire x1="46.05" y1="1.25" x2="46.1" y2="1.3" width="1.27" layer="1"/>
 </signal>
@@
 <contactref element="D3" pad="CATHODE"/>
 <contactref element="D4" pad="ANODE"/>
-<wire x1="16.95" y1="4.75" x2="30.7" y2="4.75" width="1.27" layer="1"/>
+<wire x1="16.6" y1="4.75" x2="30.35" y2="4.75" width="1.27" layer="1"/>
 </signal>
 <signal name="N$5">
 <contactref element="+L" pad="1"/>
 <contactref element="D3" pad="ANODE"/>
-<wire x1="1.9" y1="4.7" x2="14.65" y2="4.7" width="1.27" layer="1"/>
-<wire x1="14.65" y1="4.7" x2="14.7" y2="4.75" width="1.27" layer="1"/>
+<wire x1="1.9" y1="4.7" x2="13.95" y2="4.7" width="1.27" layer="1"/>
+<wire x1="13.95" y1="4.7" x2="14.35" y2="4.75" width="1.27" layer="1"/>
 </signal>
 <signal name="N$6">
 <contactref element="D4" pad="CATHODE"/>
 <contactref element="-L" pad="1"/>
-<wire x1="32.95" y1="4.75" x2="46.05" y2="4.75" width="1.27" layer="1"/>
+<wire x1="32.6" y1="4.75" x2="46.05" y2="4.75" width="1.27" layer="1"/>
 <wire x1="46.05" y1="4.75" x2="46.1" y2="4.7" width="1.27" layer="1"/>
 </signal>
