File: Hardware/ProBack_LED_backlight/3xLED_Panel.sch (EAGLE design)
At the start: 11 parts

Commit message: Updated for PCBWay of doing boards
Parts:
- removed +1: WIREPAD1,6/0,9, wirepad:2,15/1,0
- removed -1: (no value), wirepad:2,15/1,0
- removed D4, D5, D6: YUJI_2835_SMD, Yuji_LED:YUJI_2835_SMD
- +: device wirepad:2,15/1,0 -> wirepad:SMD3X2.15
- -: value (none) -> SMD3X2.15; device wirepad:2,15/1,0 -> wirepad:SMD3X2.15
Connections:
- removed net N$5: D4.CATHODE, D5.ANODE
- removed net N$6: +1.P, D4.ANODE
- removed net N$7: D5.CATHODE, D6.ANODE
- removed net N$8: -1.P, D6.CATHODE
Changed lines of the file:
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@@
 <attribute name="VER" value="1.0"/>
 </part>
-<part name="+" library="wirepad" deviceset="2,15/1,0" device="" package3d_urn="urn:adsk.eagle:package:30831/1" value="WIREPAD1,6/0,9"/>
-<part name="-" library="wirepad" deviceset="2,15/1,0" device="" package3d_urn="urn:adsk.eagle:package:30831/1"/>
+<part name="+" library="wirepad" deviceset="SMD3X2.15" device="" value="WIREPAD1,6/0,9"/>
+<part name="-" library="wirepad" deviceset="SMD3X2.15" device="" value=""/>
 <part name="D3" library="Yuji_LED" deviceset="YUJI_2835_SMD" device=""/>
-<part name="D4" library="Yuji_LED" deviceset="YUJI_2835_SMD" device=""/>
-<part name="D5" library="Yuji_LED" deviceset="YUJI_2835_SMD" device=""/>
-<part name="+1" library="wirepad" deviceset="2,15/1,0" device="" package3d_urn="urn:adsk.eagle:package:30831/1" value="WIREPAD1,6/0,9"/>
-<part name="-1" library="wirepad" deviceset="2,15/1,0" device="" package3d_urn="urn:adsk.eagle:package:30831/1"/>
-<part name="D6" library="Yuji_LED" deviceset="YUJI_2835_SMD" device=""/>
 </parts>
 <sheets>
@@
 </instance>
 <instance part="FRAME1" gate="G$1" x="0" y="0" smashed="yes"/>
-<instance part="+" gate="1" x="27.94" y="96.52" smashed="yes">
+<instance part="+" gate="G$1" x="27.94" y="96.52" smashed="yes">
 <attribute name="NAME" x="24.003" y="97.4598" size="1.778" layer="95" rot="R180"/>
 </instance>
-<instance part="-" gate="1" x="78.74" y="96.52" smashed="yes" rot="R180">
+<instance part="-" gate="G$1" x="78.74" y="96.52" smashed="yes" rot="R180">
 <attribute name="NAME" x="84.709" y="95.8342" size="1.778" layer="95"/>
 <attribute name="VALUE" x="79.883" y="99.822" size="1.778" layer="96" rot="R180"/>
@@
 <instance part="D3" gate="G$1" x="66.04" y="96.52" smashed="yes">
 <attribute name="NAME" x="60.96" y="101.092" size="1.778" layer="95"/>
-</instance>
-<instance part="D4" gate="G$1" x="40.64" y="86.36" smashed="yes">
-<attribute name="NAME" x="36.322" y="90.932" size="1.778" layer="95"/>
-</instance>
-<instance part="D5" gate="G$1" x="53.34" y="86.36" smashed="yes">
-<attribute name="NAME" x="48.26" y="90.932" size="1.778" layer="95"/>
-</instance>
-<instance part="+1" gate="1" x="27.94" y="86.36" smashed="yes">
-<attribute name="NAME" x="24.003" y="87.2998" size="1.778" layer="95" rot="R180"/>
-</instance>
-<instance part="-1" gate="1" x="78.74" y="86.36" smashed="yes" rot="R180">
-<attribute name="NAME" x="84.709" y="85.6742" size="1.778" layer="95"/>
-<attribute name="VALUE" x="79.883" y="89.662" size="1.778" layer="96" rot="R180"/>
-</instance>
-<instance part="D6" gate="G$1" x="66.04" y="86.36" smashed="yes">
-<attribute name="NAME" x="60.96" y="90.932" size="1.778" layer="95"/>
 </instance>
 </instances>
@@
 <net name="N$2" class="0">
 <segment>
-<pinref part="+" gate="1" pin="P"/>
+<pinref part="+" gate="G$1" pin="P"/>
 <pinref part="D1" gate="G$1" pin="ANODE"/>
 <wire x1="30.48" y1="96.52" x2="35.56" y2="96.52" width="0.1524" layer="91"/>
@@
 <segment>
 <pinref part="D3" gate="G$1" pin="CATHODE"/>
-<pinref part="-" gate="1" pin="P"/>
+<pinref part="-" gate="G$1" pin="P"/>
 <wire x1="68.58" y1="96.52" x2="76.2" y2="96.52" width="0.1524" layer="91"/>
-</segment>
-</net>
-<net name="N$5" class="0">
-<segment>
-<pinref part="D4" gate="G$1" pin="CATHODE"/>
-<pinref part="D5" gate="G$1" pin="ANODE"/>
-<wire x1="43.18" y1="86.36" x2="48.26" y2="86.36" width="0.1524" layer="91"/>
-</segment>
-</net>
-<net name="N$6" class="0">
-<segment>
-<pinref part="+1" gate="1" pin="P"/>
-<pinref part="D4" gate="G$1" pin="ANODE"/>
-<wire x1="30.48" y1="86.36" x2="35.56" y2="86.36" width="0.1524" layer="91"/>
-</segment>
-</net>
-<net name="N$7" class="0">
-<segment>
-<pinref part="D5" gate="G$1" pin="CATHODE"/>
-<pinref part="D6" gate="G$1" pin="ANODE"/>
-<wire x1="55.88" y1="86.36" x2="60.96" y2="86.36" width="0.1524" layer="91"/>
-</segment>
-</net>
-<net name="N$8" class="0">
-<segment>
-<pinref part="D6" gate="G$1" pin="CATHODE"/>
-<pinref part="-1" gate="1" pin="P"/>
-<wire x1="68.58" y1="86.36" x2="76.2" y2="86.36" width="0.1524" layer="91"/>
 </segment>
 </net>
@@
 will not be understood (or retained) with this version.
 </note>
-<note version="8.3" severity="warning">
-Since Version 8.3, EAGLE supports the association of 3D packages
-with devices in libraries, schematics, and board files. Those 3D
-packages will not be understood (or retained) with this version.
-</note>
 </compatibility>
