File: Hardware/ProBack_LED_backlight/LED_Driver_Separate.sch (EAGLE design)
At the start: 13 parts, among them U1 LT1937ES5

Commit message: Update boards and schematic
Other:
- note added: "R2 value select for your LEDs current I(LED): R (Ohms) = 95 mV / I(LED) mA Current value is for 60mA LEDs"
Changed lines of the file:
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@@
 <sheet>
 <plain>
+<text x="40.64" y="38.1" size="2.1844" layer="97">R2 value select for your LEDs current I(LED):
+R (Ohms) = 95 mV / I(LED) mA
+Current value is for 60mA LEDs</text>
 </plain>
 <instances>
@@
 </drawing>
 <compatibility>
+<note version="6.3" minversion="6.2.2" severity="warning">
+Since Version 6.2.2 text objects can contain more than one line,
+which will not be processed correctly with this version.
+</note>
 <note version="8.2" severity="warning">
 Since Version 8.2, EAGLE supports online libraries. The ids

Commit message: Updated schematic and boards
Parts:
- D2: value DIODE-ZENER -> MM5Z20; device SparkFun-DiscreteSemi:DIODE-ZENER -> SparkFun-DiscreteSemi:DIODE-ZENERSOD-523Z
Other:
- note added: "MM5Z20"
- note added: "Zener - current DZ9F20S92 R2 value select for your LEDs current I(LED): R (Ohms) = 95 mV / I(LED) mA. Preset values: - 1.6 Ohm - 60mA LEDs - 2.1 Ohm - 45mA LEDs - 2.37 Ohm - 40mA LEDs - 2.71 Ohm - 35mA LEDs - 3.16 Ohm - 30mA LEDs"
- note removed: "R2 value select for your LEDs current I(LED): R (Ohms) = 95 mV / I(LED) mA Current value is for 60mA LEDs"
Changed lines of the file:
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@@
 <part name="L1" library="SparkFun-Passives" deviceset="INDUCTOR" device="1210" value="22uH"/>
 <part name="R2" library="rcl" library_urn="urn:adsk.eagle:library:334" deviceset="R-EU_" device="M1206" package3d_urn="urn:adsk.eagle:package:23566/2" value="1.6"/>
-<part name="D2" library="SparkFun-DiscreteSemi" deviceset="DIODE-ZENER" device=""/>
+<part name="D2" library="SparkFun-DiscreteSemi" deviceset="DIODE-ZENER" device="SOD-523Z" value="MM5Z20"/>
 <part name="P+1" library="Spectron2" deviceset="3.3V" device=""/>
 <part name="FRAME1" library="SparkFun-Aesthetics" deviceset="FRAME-LEDGER" device="">
@@
 <sheet>
 <plain>
-<text x="40.64" y="38.1" size="2.1844" layer="97">R2 value select for your LEDs current I(LED):
-R (Ohms) = 95 mV / I(LED) mA
-Current value is for 60mA LEDs</text>
+<text x="99.06" y="48.26" size="2.1844" layer="97" rot="R180">Zener - current DZ9F20S92
+R2 value select for your LEDs current I(LED):
+R (Ohms) = 95 mV / I(LED) mA. Preset values:
+ - 1.6 Ohm  - 60mA LEDs
+ - 2.1 Ohm  - 45mA LEDs
+ - 2.37 Ohm - 40mA LEDs
+ - 2.71 Ohm - 35mA LEDs
+ - 3.16 Ohm - 30mA LEDs
+</text>
+<text x="73.66" y="81.28" size="1.778" layer="96">MM5Z20</text>
 </plain>
 <instances>

Commit message: Update description
Other:
- note added: "R2 value select for your LEDs current I(LED): R (Ohms) = 95 mV / I(LED) mA. Preset values: - 1.6 Ohm - 60mA LEDs - 2.1 Ohm - 45mA LEDs - 2.37 Ohm - 40mA LEDs - 2.71 Ohm - 35mA LEDs - 3.16 Ohm - 30mA LEDs"
- note removed: "Zener - current DZ9F20S92 R2 value select for your LEDs current I(LED): R (Ohms) = 95 mV / I(LED) mA. Preset values: - 1.6 Ohm - 60mA LEDs - 2.1 Ohm - 45mA LEDs - 2.37 Ohm - 40mA LEDs - 2.71 Ohm - 35mA LEDs - 3.16 Ohm - 30mA LEDs"
Changed lines of the file:
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@@
 <sheet>
 <plain>
-<text x="99.06" y="48.26" size="2.1844" layer="97" rot="R180">Zener - current DZ9F20S92
-R2 value select for your LEDs current I(LED):
+<text x="99.06" y="48.26" size="2.1844" layer="97" rot="R180">R2 value select for your LEDs current I(LED):
 R (Ohms) = 95 mV / I(LED) mA. Preset values:
  - 1.6 Ohm  - 60mA LEDs
